File: Panel/noisebells_panel/noisebells_panel.kicad_pcb (KiCad board)
At the start: 2 copper layers, 100 x 200 mm, 18 parts

Commit message: Final design for first run
Other:
- board text added: "Panel design Rich Holmes Sep 2020"
- board text removed: "Panel design: Rich Holmes 9/2020"
