File: jackboard4/jackboard4.kicad_pcb (KiCad board)
At the start: 2 copper layers, 96 x 25 mm, 6 parts, among them J1 AudioJack2_SwitchT, J2 AudioJack2_SwitchT, J3 Conn_01x05, J4 AudioJack2_SwitchT, J5 AudioJack2_SwitchT

Commit message: Final design for first run
Parts:
- added G***: LOGO, jackboard4:noisebells_holes, B.Cu at (205.4, 120.1)
