File: noisebells/noisebells.kicad_pcb (KiCad board)
At the start: 2 copper layers, 96 x 144 mm, 50 parts, among them J1 Synth_power_2x5, J2 Conn_01x05, Q1 2N3904, Q2 2N3904, SW1 SW_DPDT_x2, SW2 SW_DPDT_x2, U1 40106, U2 4070, U3 4066

Commit message: Final design for first run
Parts:
- removed the G*** at (207.0, 142.9)
- added G***: LOGO, noisebells_panel:noisebells_holes, B.Cu at (207.0, 143.0)
- RV1, RV2, RV3, RV4, RV5, RV6, RV7, RV8: footprint ao_tht:Potentiometer_Alpha_RD901F-40-00D_Single_Vertical_CircularHoles -> ao_tht:Potentiometer_Alpha_RD901F-40-00D_Single_Vertical_CircularHoles_centered
- moved RV1 7.91 mm to (242.0, 72.9)
- moved RV2 7.91 mm to (242.0, 107.9)
- moved RV3 7.91 mm to (207.0, 72.9)
- moved RV5 7.91 mm to (207.0, 107.9)
- moved RV6 7.91 mm to (172.0, 107.9)
- moved RV7 7.91 mm to (242.0, 177.9)
- moved RV8 7.91 mm to (189.5, 177.9)
- moved RV4 7.81 mm to (172.0, 73.0)
- moved SW2 0.10 mm to (189.5, 148.0)
- moved SW1 0.10 mm to (242.0, 148.0)
